File: Starbie/Starbie.kicad_pcb (KiCad board)
At the start: 2 copper layers, 80 x 70 mm, 7 parts, among them J1 Conn_01x04_Pin, J2 Conn_01x08_Pin, SW1 SW_Push, SW3 SW_Push, U1 XIAO-ESP32-C3-SMD, U2 DHT11

Commit message: Move XIAO to board edge with USB facing out, reroute, add board image
Parts:
- moved U1 18.6 mm to (177.6, 95.6), turned to -90 degrees
Routing:
- net GND: track 28.2 -> 1.83 mm
- net +3.3V: track 99.4 -> 75.7 mm, vias 0 -> 1
- net /GPIO2: track 50.2 -> 58.7 mm, vias 0 -> 1
- net /SCL: track 32.3 -> 39.6 mm
- net /SDA: track 35.9 -> 41.1 mm, vias 0 -> 1
- net /GPIO3: track 56.4 -> 52.9 mm
- net /DHT11_DATA: track 40.6 -> 38.9 mm, vias 0 -> 1
